File: artemis.kicad_sch (KiCad schematic)
At the start: 26 parts, among them SW1 RESET, U1 Sparkfun Artemis, Y1 32.768kHz

Commit message: Revision B
Fixed SWDIO/SWDCK
Relabeled ADC Caps to 10nF
Relabelled LORA reset line to active low
Minor silkscreen tweaks
Connections:
- net SWDCK: now also J_DEBUG0.4 (Pin_4); no longer J_DEBUG0.2 (Pin_2)
- net SWDIO: now also J_DEBUG0.2 (Pin_2); no longer J_DEBUG0.4 (Pin_4)
- net LORA_RST renamed LORA_nRST
Other:
- title: (none) -> Cathodic Protection Sensor Mk1
Changed lines of the file:
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@@
 	(generator_version "8.0")
 	(paper "A4")
+	(title_block
+		(title "Cathodic Protection Sensor Mk1")
+		(date "2024-06-10")
+		(rev "B")
+	)
 	(bus_alias "SPI"
 		(members "SCK" "MISO" "MOSI" "nCE[0..3]")
@@
 		)
 	)
-	(text_box "ADC Notes:\n\nADCs have a ~4pF sampling capacitor, may underestimate for high-impedance\nsources, may need decoupling cap (~0.1uF should be plenty?)\nhttps://forum.sparkfun.com/viewtopic.php?t=54907\n\nADCs measure up to internal 1.5V or 2V reference, may need dividers to measure higher voltages"
+	(text_box "ADC Notes:\n\nADCs have a ~4pF sampling capacitor, may underestimate for high-impedance\nsources, may need decoupling cap (1nF should be plenty, and with 100kOhm gives\ntime constant = 0.1ms)\nhttps://forum.sparkfun.com/viewtopic.php?t=54907\n\nADCs measure up to internal 1.5V or 2V reference, may need dividers to measure higher voltages"
 		(exclude_from_sim no)
 		(at 19.05 101.6 0)
@@
 	)
 	(label "SWDIO"
-		(at 276.86 58.42 180)
+		(at 276.86 55.88 180)
 		(fields_autoplaced yes)
 		(effects
@@
 	)
 	(label "SWDCK"
-		(at 276.86 55.88 180)
+		(at 276.86 58.42 180)
 		(fields_autoplaced yes)
 		(effects
@@
 		)
 	)
-	(hierarchical_label "LORA_RST"
+	(hierarchical_label "LORA_nRST"
 		(shape input)
 		(at 181.61 109.22 0)
