File: cpm_proj.kicad_sch (KiCad schematic)
At the start: 28 parts, among them J11 USB_C_Receptacle_USB2.0, U4 TPS22860, U5 LD1117AV33_TO220

Commit message: Revision B
Fixed SWDIO/SWDCK
Relabeled ADC Caps to 10nF
Relabelled LORA reset line to active low
Minor silkscreen tweaks
Parts:
- added H1, H2, H3, H4: MountingHole, MountingHole:MountingHole_3.5mm, symbol Mechanical:MountingHole
Connections:
- no-connect marks 7 -> 12
Other:
- sheet artemis ports: added LORA_nRST; removed LORA_RST
- title: (none) -> Cathodic Protection Sensor Mk1
