File: power.kicad_sch (KiCad schematic)
At the start: 29 parts, among them U2 ADP5091

Commit message: Revision B
Fixed SWDIO/SWDCK
Relabeled ADC Caps to 10nF
Relabelled LORA reset line to active low
Minor silkscreen tweaks
Other:
- title: (none) -> Cathodic Protection Sensor Mk1
Changed lines of the file:
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@@
 	(generator_version "8.0")
 	(paper "A4")
+	(title_block
+		(title "Cathodic Protection Sensor Mk1")
+		(date "2024-06-10")
+		(rev "B")
+	)
 	(junction
 		(at 224.79 134.62)
